File: circuit/hub/hub.kicad_pcb (KiCad board)
At the start: 2 copper layers, 46.5 x 34 mm, 57 parts, among them J1 Host-IMU, J2 Dev1, J3 Dev5, J4 Dev7, J5 Dev6, J6 Dev2, J7 Dev4, U1 NJM2884U1-33, U2 USB2517, X1 SG-210STF

Commit message: update circuits
Parts:
- removed the D1 at (149.7, 108.6)
- removed D3, D4, D5, D6, D7, D8, D9: KM-23YSGC, TO_SOT_Packages_SMD:SOT-23
- removed R11, R12, R13, R14, R15, R16, R17, R18, R19, R20, R21, R22, R23, R24: 1k, Resistors_SMD:R_0603
- removed the R2 at (148.1, 112.4)
- added REF**: MountingHole_2.2mm_M2_Pad_Via, Mounting_Holes:MountingHole_2.2mm_M2_Pad_Via, F.Cu at (152.5, 118.8)
- added REF**: MountingHole_2.2mm_M2_Pad_Via, Mounting_Holes:MountingHole_2.2mm_M2_Pad_Via, F.Cu at (128.0, 118.8)
- added REF**: MountingHole_2.2mm_M2_Pad_Via, Mounting_Holes:MountingHole_2.2mm_M2_Pad_Via, F.Cu at (128.0, 89.3)
- added REF**: MountingHole_2.2mm_M2_Pad_Via, Mounting_Holes:MountingHole_2.2mm_M2_Pad_Via, F.Cu at (152.5, 89.3)
- moved J6 11.5 mm to (158.8, 112.2)
- moved J3 11.5 mm to (158.8, 101.9)
- moved J7 11.5 mm to (163.9, 112.2)
- moved J2 11.5 mm to (163.8, 101.9)
- moved J5 11.3 mm to (129.5, 94.6), turned to 270 degrees
- moved J4 10.8 mm to (140.1, 90.6), turned to 180 degrees
- moved C3 7.80 mm to (145.7, 110.4), turned to 0 degrees
- moved R7 6.18 mm to (152.8, 110.4)
- moved C1 4.80 mm to (142.6, 114.6), turned to 90 degrees
- moved R2 4.27 mm to (137.6, 113.1)
- moved R3 4.27 mm to (139.2, 113.1)
- moved R8 4.27 mm to (136.0, 113.1)
- moved R5 4.27 mm to (134.3, 113.1)
- moved C12 3.93 mm to (145.1, 101.0)
- moved C2 3.79 mm to (148.6, 100.7)
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- renumbered D2 to D1, J6 to J3, J7 to J4, J3 to J5, J5 to J6, J4 to J7, R3 to R2, R4 to R3, R5 to R4, R6 to R5, R7 to R6, R8 to R7, R9 to R8, R10 to R9
Connections:
- U2 pad 1: /Dev7D- -> /Dev1D-
- U2 pad 11: /Dev3D- -> /Dev5D-
- U2 pad 12: /Dev3D+ -> /Dev5D+
- U2 pad 14: /LED_YELLOW7 -> (no net)
- U2 pad 15: /LED_GREEN1 -> (no net)
- U2 pad 16: /LED_YELLOW6 -> (no net)
- U2 pad 17: /LED_GREEN2 -> (no net)
- U2 pad 18: /LED_YELLOW5 -> (no net)
- U2 pad 2: /Dev7D+ -> /Dev1D+
- U2 pad 3: /Dev6D- -> /Dev2D-
- U2 pad 31: /LED_GREEN3 -> (no net)
- U2 pad 32: /LED_YELLOW4 -> (no net)
- U2 pad 33: /LED_GREEN4 -> (no net)
- U2 pad 34: /LED_YELLOW3 -> (no net)
- U2 pad 4: /Dev6D+ -> /Dev2D+
- U2 pad 47: /LED_GREEN5 -> (no net)
- U2 pad 48: /LED_YELLOW2 -> (no net)
- U2 pad 49: /LED_GREEN6 -> (no net)
- U2 pad 50: /LED_YELLOW1 -> (no net)
- U2 pad 51: /LED_GREEN7 -> (no net)
- U2 pad 53: /Dev2D- -> /Dev6D-
- U2 pad 54: /Dev2D+ -> /Dev6D+
- U2 pad 55: /Dev1D- -> /Dev7D-
- U2 pad 56: /Dev1D+ -> /Dev7D+
- U2 pad 6: /Dev5D- -> /Dev3D-
- U2 pad 7: /Dev5D+ -> /Dev3D+
Routing:
- net GND: track 301.1 -> 511.1 mm, vias 82 -> 199
- net /LED_GREEN7: track 74.5 -> 0.00 mm, vias 6 -> 0
- net /LED_GREEN6: track 70.4 -> 0.00 mm, vias 4 -> 0
- net /LED_YELLOW1: track 68.0 -> 0.00 mm, vias 6 -> 0
- net /LED_GREEN4: track 61.2 -> 0.00 mm, vias 4 -> 0
- net /LED_YELLOW3: track 55.8 -> 0.00 mm, vias 4 -> 0
- net /LED_GREEN2: track 52.7 -> 0.00 mm, vias 4 -> 0
- net /LED_GREEN5: track 47.0 -> 0.00 mm, vias 4 -> 0
- net /LED_YELLOW4: track 41.7 -> 0.00 mm, vias 2 -> 0
- net /LED_YELLOW5: track 39.9 -> 0.00 mm, vias 4 -> 0
- net /LED_GREEN3: track 36.5 -> 0.00 mm, vias 2 -> 0
- net Net-(D3-Pad2): track 35.0 -> 0.00 mm, vias 4 -> 0
- net /LED_GREEN1: track 32.3 -> 0.00 mm, vias 4 -> 0
- net /LED_YELLOW7: track 23.6 -> 0.00 mm, vias 2 -> 0
- net /LED_YELLOW6: track 22.8 -> 0.00 mm, vias 2 -> 0
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Other:
- outline, holes or cut-outs redrawn
